File: Power_supply.kicad_sch (KiCad schematic)
At the start: 22 parts, among them J10 USB_C_Receptacle, U4 AMS1117-5.0

Commit message: Inclusão dos arquivos de fabricação para 1ª cotação
Parts:
- R?: value 120k -> 110k
Changed lines of the file:
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@@
       (effects (font (size 1.27 1.27)) (justify left))
     )
-    (property "Value" "120k" (at 160.02 154.305 0)
+    (property "Value" "110k" (at 160.02 154.305 0)
       (effects (font (size 1.27 1.27)) (justify left))
     )
@@
       (effects (font (size 1.27 1.27)) hide)
     )
-    (property "Description" "Chip Resistor 169k ±0,1% 1/8W ±25ppm/ºC 0805_2012Metric" (at 158.75 164.465 0)
+    (property "Description" "Chip Resistor 110k ±0,1% 1/8W ±25ppm/ºC 0805_2012Metric" (at 158.75 164.465 0)
       (effects (font (size 1.27 1.27)) hide)
     )
