File: User_interface.kicad_sch (KiCad schematic)
At the start: 32 parts, among them J11 PinHeader_01x02_P2.54mm_Verti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, J12 PinHeader_01x02_P2.54mm_Verti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, J13 PinHeader_01x02_P2.54mm_Verti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, J14 PinHeader_01x02_P2.54mm_Verti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, U7 TMP126

Commit message: Inclusão dos arquivos de fabricação para 1ª cotação
Other:
- moved on the sheet: J11, J14, R?, SW?
