File: data_logger.kicad_pcb (KiCad board)
At the start: 2 copper layers, 120.2 x 74.4 mm, 89 parts, among them J1 PinHeader_01x01_P2.54mm_Verti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, J10 USB_C_Receptacle, J11 PinHeader_01x02_P2.54mm_Verti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, J12 PinHeader_01x02_P2.54mm_Verti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, J13 PinHeader_01x02_P2.54mm_Verti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, J14 PinHeader_01x02_P2.54mm_Verti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, J15 Micro_SD_Card_Det, J2 PinHeader_01x01_P2.54mm_Verti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, J3 Conn_01x03, J4 PinHeader_01x06_P2.54mm_Verti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

Commit message: Inclusão dos arquivos de fabricação para 1ª cotação
Routing:
- net +5V: track 268.9 -> 270.6 mm
- net GND: vias 213 -> 217
Changed lines of the file:
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@@
   (via (at 87.204546 69.7) (size 0.5) (drill 0.25) (layers "F.Cu" "B.Cu") (free) (net 2))
   (via (at 85.612728 77.436664) (size 0.5) (drill 0.25) (layers "F.Cu" "B.Cu") (free) (net 2))
+  (via (at 150.975 66.233334) (size 0.5) (drill 0.25) (layers "F.Cu" "B.Cu") (free) (net 2))
   (via (at 101.530908 72.21) (size 0.5) (drill 0.25) (layers "F.Cu" "B.Cu") (free) (net 2))
   (via (at 101.530908 68.39) (size 0.5) (drill 0.25) (layers "F.Cu" "B.Cu") (free) (net 2))
@@
   (via (at 103.122728 64.46) (size 0.5) (drill 0.25) (layers "F.Cu" "B.Cu") (free) (net 2))
   (via (at 109.94 69.41) (size 0.5) (drill 0.25) (layers "F.Cu" "B.Cu") (free) (net 2))
+  (via (at 150.975 68.875) (size 0.5) (drill 0.25) (layers "F.Cu" "B.Cu") (free) (net 2))
   (via (at 95.163636 63.15) (size 0.5) (drill 0.25) (layers "F.Cu" "B.Cu") (free) (net 2))
   (via (at 99.93909 78.74333) (size 0.5) (drill 0.25) (layers "F.Cu" "B.Cu") (free) (net 2))
@@
   (via (at 101.530908 73.516666) (size 0.5) (drill 0.25) (layers "F.Cu" "B.Cu") (free) (net 2))
   (via (at 87.204546 68.39) (size 0.5) (drill 0.25) (layers "F.Cu" "B.Cu") (free) (net 2))
+  (via (at 150.975 63.591668) (size 0.5) (drill 0.25) (layers "F.Cu" "B.Cu") (free) (net 2))
   (via (at 101.530908 69.7) (size 0.5) (drill 0.25) (layers "F.Cu" "B.Cu") (free) (net 2))
   (via (at 117.99 71.56) (size 0.5) (drill 0.25) (layers "F.Cu" "B.Cu") (free) (net 2))
@@
   (via (at 88.49 91.26) (size 0.5) (drill 0.25) (layers "F.Cu" "B.Cu") (free) (net 2))
   (via (at 96.755454 80.05) (size 0.5) (drill 0.25) (layers "F.Cu" "B.Cu") (free) (net 2))
+  (via (at 150.975 71.516668) (size 0.5) (drill 0.25) (layers "F.Cu" "B.Cu") (free) (net 2))
   (via (at 101.530908 64.46) (size 0.5) (drill 0.25) (layers "F.Cu" "B.Cu") (free) (net 2))
   (via (at 91.98 78.74333) (size 0.5) (drill 0.25) (layers "F.Cu" "B.Cu") (free) (net 2))
@@
   (segment (start 175.79 71.66) (end 175.79 70.86) (width 0.8) (layer "B.Cu") (net 5))
   (segment (start 162.99 121.06) (end 162.99 121.86) (width 0.8) (layer "B.Cu") (net 5))
-  (segment (start 164.57 102.58) (end 162.99 104.16) (width 0.8) (layer "B.Cu") (net 5))
-  (segment (start 169.166 102.58) (end 164.57 102.58) (width 0.8) (layer "B.Cu") (net 5))
+  (segment (start 164.32 101.18) (end 162.125 103.375) (width 0.8) (layer "B.Cu") (net 5))
+  (segment (start 162.125 103.375) (end 162.125 120.195) (width 0.8) (layer "B.Cu") (net 5))
   (segment (start 189.79 98.76) (end 187.13 96.1) (width 0.8) (layer "B.Cu") (net 5))
   (segment (start 187.13 96.1) (end 185.806 96.1) (width 0.8) (layer "B.Cu") (net 5))
   (segment (start 175.79 86.084) (end 175.79 71.66) (width 0.8) (layer "B.Cu") (net 5))
-  (segment (start 170.566 101.18) (end 169.166 102.58) (width 0.8) (layer "B.Cu") (net 5))
+  (segment (start 162.125 120.195) (end 162.99 121.06) (width 0.8) (layer "B.Cu") (net 5))
   (segment (start 161.79 129.96) (end 185.19 129.96) (width 0.8) (layer "B.Cu") (net 5))
   (segment (start 185.19 129.96) (end 189.79 125.36) (width 0.8) (layer "B.Cu") (net 5))
@@
   (segment (start 160.785 130.965) (end 161.79 129.96) (width 0.8) (layer "B.Cu") (net 5))
   (segment (start 185.806 96.1) (end 175.79 86.084) (width 0.8) (layer "B.Cu") (net 5))
-  (segment (start 162.99 104.16) (end 162.99 121.06) (width 0.8) (layer "B.Cu") (net 5))
+  (segment (start 170.566 101.18) (end 164.32 101.18) (width 0.8) (layer "B.Cu") (net 5))
   (segment (start 123.29 75.21) (end 126.42 75.21) (width 0.4) (layer "F.Cu") (net 6))
   (segment (start 170.415348 108.649348) (end 170.566 108.8) (width 0.2) (layer "F.Cu") (net 7))
@@
   (segment (start 101.99 88.82) (end 106.89 93.72) (width 0.2) (layer "F.Cu") (net 22))
   (segment (start 106.89 85.52) (end 110.39 85.52) (width 0.2) (layer "F.Cu") (net 23))
+  (segment (start 111.248 123.798) (end 111.248 124.71) (width 0.4) (layer "F.Cu") (net 24))
+  (segment (start 109.12 121.86) (end 109.31 121.86) (width 0.4) (layer "F.Cu") (net 24))
   (segment (start 105.99 128.97) (end 105.99 129.580406) (width 0.3) (layer "F.Cu") (net 24))
   (segment (start 105.99 129.580406) (end 106.175 129.765406) (width 0.3) (layer "F.Cu") (net 24))
-  (segment (start 109.5 121.86) (end 111.248 123.608) (width 0.4) (layer "F.Cu") (net 24))
-  (segment (start 111.248 123.608) (end 111.248 124.71) (width 0.4) (layer "F.Cu") (net 24))
   (segment (start 106.848 130.46) (end 109.910406 130.46) (width 0.3) (layer "F.Cu") (net 24))
   (segment (start 106.175 129.765406) (end 106.175 129.787) (width 0.3) (layer "F.Cu") (net 24))
   (segment (start 110.79 129.580406) (end 110.79 128.97) (width 0.3) (layer "F.Cu") (net 24))
   (segment (start 109.910406 130.46) (end 110.79 129.580406) (width 0.3) (layer "F.Cu") (net 24))
-  (segment (start 109.12 121.86) (end 109.5 121.86) (width 0.4) (layer "F.Cu") (net 24))
+  (segment (start 109.31 121.86) (end 111.248 123.798) (width 0.4) (layer "F.Cu") (net 24))
   (segment (start 110.79 125.168) (end 111.248 124.71) (width 0.4) (layer "F.Cu") (net 24))
   (segment (start 110.79 128.97) (end 110.79 125.168) (width 0.4) (layer "F.Cu") (net 24))
@@
   (segment (start 110.81 118.585) (end 110.835 118.56) (width 0.4) (layer "F.Cu") (net 33))
   (segment (start 109.158423 116.158423) (end 109.31 116.31) (width 0.4) (layer "F.Cu") (net 33))
-  (segment (start 110.835 116.147501) (end 110.847501 116.135) (width 0.4) (layer "F.Cu") (net 33))
   (segment (start 108.14 128.97) (end 108.14 129.795) (width 0.2) (layer "F.Cu") (net 34))
   (segment (start 107.628 127.34) (end 108.14 127.852) (width 0.2) (layer "F.Cu") (net 34))
@@
     (polygon
       (pts
-        (xy 111.12 115.9)
-        (xy 109.98 115.87)
-        (xy 109.68 115.66)
-        (xy 104.8 115.66)
-        (xy 102.13 117.81)
-        (xy 102.23 119.07)
-        (xy 104.06 119.02)
-        (xy 108.8 118.38)
-        (xy 109.91 118.41)
-        (xy 110.11 118.7)
-        (xy 110.57 121.93)
-        (xy 111.96 121.93)
-        (xy 111.46 119.25)
-        (xy 111.46 117.79)
-        (xy 111.12 115.89)
+        (xy 102.15 117.7)
+        (xy 102.15 118.975)
+        (xy 102.175 119)
+        (xy 108.125 119)
+        (xy 108.7 118.425)
+        (xy 109.575 118.425)
+        (xy 110.325 119.175)
+        (xy 110.325 122.1)
+        (xy 112.05 122.1)
+        (xy 112.225 121.925)
+        (xy 112.225 120.075)
+        (xy 111.575 119.425)
+        (xy 111.575 117.9375)
+        (xy 111.410252 116.523805)
+        (xy 111.135202 116.010202)
+        (xy 110.9 115.775)
+        (xy 109.275 115.525)
+        (xy 104.939381 116.139381)
       )
     )
@@
     (polygon
       (pts
-        (xy 112.56 115.97)
-        (xy 112.11 117.91)
-        (xy 112.11 119.34)
-        (xy 113.44 119.34)
-        (xy 114.4 119.04)
-        (xy 115.51 119.04)
-        (xy 116.75 119.64)
-        (xy 118.78 119.82)
-        (xy 119.91 122.07)
-        (xy 121.29 122.07)
-        (xy 121.28 119.16)
-        (xy 119.93 119.14)
-        (xy 119.83 119.05)
-        (xy 119.83 118.14)
-        (xy 121.3 118.06)
-        (xy 121.27 117.17)
-        (xy 113.2 115.9)
-        (xy 112.55 115.97)
+        (xy 112.525 117.4)
+        (xy 111.95 117.975)
+        (xy 111.95 119.2)
+        (xy 112.325 119.575)
+        (xy 113.75 119.575)
+        (xy 114.275 119.05)
+        (xy 116.1 119.05)
+        (xy 117.25 120.2)
+        (xy 119.8 122.05)
+        (xy 121.25 122.05)
+        (xy 121.5 120.2)
+        (xy 121.5 119.175)
+        (xy 121.45 119.125)
+        (xy 119.775 119.125)
+        (xy 119.75 119.15)
+        (xy 119.725 119.125)
+        (xy 119.725 118.175)
+        (xy 119.775 118.125)
+        (xy 121.45 118.125)
+        (xy 121.45 117.075)
+        (xy 121.425 117.05)
+        (xy 116 117.05)
+        (xy 115.9 117.15)
+        (xy 114.75 117.15)
+        (xy 113.475 115.875)
+        (xy 112.525 115.875)
       )
     )
